File: pi_poe_hat/pi_poe_hat.kicad_pcb (KiCad board)
At the start: 2 copper layers, 3 parts, among them J1 8P8C_LED_Shielded, U1 PD70X01

Commit message: PD done???
Parts:
- added D1: ABS10, Diode_SMD:Diode_Bridge_Diotec_ABS, F.Cu at (60.5, 60.0)
- added D2: ABS10, Diode_SMD:Diode_Bridge_Diotec_ABS, F.Cu at (60.5, 66.6)
- added J2: ENABLE, Connector_PinHeader_2.54mm:PinHeader_1x03_P2.54mm_Vertical, F.Cu at (67.1, 59.1)
Connections:
- J1 pad 1: unconnected-(J1-Pad1) -> Net-(TR1-MX1+)
- J1 pad 2: unconnected-(J1-Pad2) -> Net-(TR1-MX1-)
- J1 pad 3: unconnected-(J1-Pad3) -> Net-(TR1-MX2+)
- J1 pad 4: unconnected-(J1-Pad4) -> Net-(TR1-MX3+)
- J1 pad 5: unconnected-(J1-Pad5) -> Net-(TR1-MX3-)
- J1 pad 6: unconnected-(J1-Pad6) -> Net-(TR1-MX2-)
- J1 pad 7: unconnected-(J1-Pad7) -> Net-(TR1-MX4+)
- J1 pad 8: unconnected-(J1-Pad8) -> Net-(TR1-MX4-)
- J1 pad SH: unconnected-(J1-PadSH) -> /VPN_IN
- TR1 pad 11: unconnected-(TR1-TD4+-Pad11) -> D4+
- TR1 pad 12: unconnected-(TR1-TD4--Pad12) -> D4-
- TR1 pad 13: unconnected-(TR1-MX4--Pad13) -> Net-(TR1-MX4-)
- TR1 pad 14: unconnected-(TR1-MX4+-Pad14) -> Net-(TR1-MX4+)
- TR1 pad 15: unconnected-(TR1-MCT4-Pad15) -> PoE+_1
- TR1 pad 16: unconnected-(TR1-MX3--Pad16) -> Net-(TR1-MX3-)
- TR1 pad 17: unconnected-(TR1-MX3+-Pad17) -> Net-(TR1-MX3+)
- TR1 pad 18: unconnected-(TR1-MCT3-Pad18) -> PoE-_1
- TR1 pad 19: unconnected-(TR1-MX2--Pad19) -> Net-(TR1-MX2-)
- TR1 pad 2: unconnected-(TR1-TD1+-Pad2) -> D1+
- TR1 pad 20: unconnected-(TR1-MX2+-Pad20) -> Net-(TR1-MX2+)
- TR1 pad 21: unconnected-(TR1-MCT2-Pad21) -> PoE+_2
- TR1 pad 22: unconnected-(TR1-MX1--Pad22) -> Net-(TR1-MX1-)
- TR1 pad 23: unconnected-(TR1-MX1+-Pad23) -> Net-(TR1-MX1+)
- TR1 pad 24: unconnected-(TR1-MCT1-Pad24) -> PoE-_2
- TR1 pad 3: unconnected-(TR1-TD1--Pad3) -> D1-
- TR1 pad 5: unconnected-(TR1-TD2+-Pad5) -> D2+
- TR1 pad 6: unconnected-(TR1-TD2--Pad6) -> D2-
- TR1 pad 8: unconnected-(TR1-TD3+-Pad8) -> D3+
- TR1 pad 9: unconnected-(TR1-TD3--Pad9) -> D3-
- U1 pad 1: unconnected-(U1-RDET-Pad1) -> Net-(U1-RDET)
- U1 pad 10: unconnected-(U1-ENABLE-Pad10) -> /EN
- U1 pad 11: unconnected-(U1-VINS-Pad11) -> /VINS
- U1 pad 12: unconnected-(U1-HYST-Pad12) -> /HYST
- U1 pad 13: unconnected-(U1-SYNC-Pad13) -> GND
- U1 pad 14: unconnected-(U1-RFREQ-Pad14) -> Net-(U1-RFREQ)
- U1 pad 15: unconnected-(U1-SS-Pad15) -> Net-(U1-SS)
- U1 pad 16: unconnected-(U1-RCLP-Pad16) -> Net-(U1-RCLP)
- U1 pad 17: unconnected-(U1-VSN-Pad17) -> /VL
- U1 pad 18: unconnected-(U1-VSP-Pad18) -> GND
- U1 pad 19: unconnected-(U1-COMP-Pad19) -> /FB
- U1 pad 2: unconnected-(U1-PGOOD-Pad2) -> PGOOD
- U1 pad 21: unconnected-(U1-FB-Pad21) -> /FB
- U1 pad 22: unconnected-(U1-GND-Pad22) -> GND
- U1 pad 23: unconnected-(U1-VL-Pad23) -> /VL
- U1 pad 25: unconnected-(U1-PGND-Pad25) -> GND
- U1 pad 26: unconnected-(U1-CSN-Pad26) -> GND
- U1 pad 29: unconnected-(U1-VH-Pad29) -> Net-(U1-VH)
- U1 pad 3: unconnected-(U1-RREF-Pad3) -> Net-(U1-RREF)
- U1 pad 30: unconnected-(U1-VCC-Pad30) -> VCC
- U1 pad 31: unconnected-(U1-VAUX-Pad31) -> Net-(U1-VAUX)
- U1 pad 32: unconnected-(U1-VPP-Pad32) -> VCC
- U1 pad 4: unconnected-(U1-RCLASS-Pad4) -> Net-(U1-RCLASS)
- U1 pad 5: unconnected-(U1-VPN_IN-Pad5) -> /VPN_IN
- U1 pad 7: unconnected-(U1-NC/AT_FLAG-Pad7) -> AT_FLAG
- U1 pad 8: unconnected-(U1-VPN_OUT-Pad8) -> GND

Commit message: done?
Parts:
- removed J2: ENABLE, Connector_PinHeader_2.54mm:PinHeader_1x03_P2.54mm_Vertical
- removed TR1: SM51589PEL, Transformer_SMD:Transformer_Ethernet_Bourns_PT61020EL
- removed U1: PD70X01, Package_DFN_QFN:QFN-32-1EP_5x5mm_P0.5mm_EP3.3x3.3mm_ThermalVias
- added C1: 1uF, Capacitor_SMD:C_0603_1608Metric_Pad1.08x0.95mm_HandSolder, F.Cu at (125.1, 42.9)
- added C10: 0.1uF, Capacitor_SMD:C_0603_1608Metric_Pad1.08x0.95mm_HandSolder, F.Cu at (125.1, 55.4)
- added C11: 0.1uF, Capacitor_SMD:C_0603_1608Metric_Pad1.08x0.95mm_HandSolder, F.Cu at (125.1, 57.9)
- added C12: 0.1uF, Capacitor_SMD:C_0603_1608Metric_Pad1.08x0.95mm_HandSolder, F.Cu at (129.4, 42.9)
- added C13: 47uF, Capacitor_SMD:C_1210_3225Metric_Pad1.33x2.70mm_HandSolder, F.Cu at (143.3, 43.7)
- added C14: 47uF, Capacitor_SMD:C_1210_3225Metric_Pad1.33x2.70mm_HandSolder, F.Cu at (143.3, 48.0)
- added C15: 470uF/16V, Capacitor_THT:CP_Radial_D10.0mm_P5.00mm, F.Cu at (117.0, 26.2)
- added C17: 2.2uF/100V, Capacitor_SMD:C_1210_3225Metric_Pad1.33x2.70mm_HandSolder, F.Cu at (143.3, 52.2)
- added C18: 2.2uF/100V, Capacitor_SMD:C_1210_3225Metric_Pad1.33x2.70mm_HandSolder, F.Cu at (143.3, 56.5)
- added C19: 47uf/100V, Capacitor_THT:CP_Radial_D8.0mm_P3.50mm, F.Cu at (54.5, 61.5)
- added C2: 27pF, Capacitor_SMD:C_0603_1608Metric_Pad1.08x0.95mm_HandSolder, F.Cu at (125.1, 45.4)
- added C20: 0.1Uf, Capacitor_SMD:C_0603_1608Metric_Pad1.08x0.95mm_HandSolder, F.Cu at (129.4, 45.4)
- added C21: 1uF, Capacitor_SMD:C_0603_1608Metric_Pad1.08x0.95mm_HandSolder, F.Cu at (129.4, 47.9)
- added C22: 4.7uF, Capacitor_SMD:C_0805_2012Metric_Pad1.18x1.45mm_HandSolder, F.Cu at (158.5, 33.6)
- added C23: 0.1Uf, Capacitor_SMD:C_0603_1608Metric_Pad1.08x0.95mm_HandSolder, F.Cu at (129.4, 50.4)
- added C24: 1uF, Capacitor_SMD:C_0603_1608Metric_Pad1.08x0.95mm_HandSolder, F.Cu at (129.4, 52.9)
- added C25: 0.1uF, Capacitor_SMD:C_0603_1608Metric_Pad1.08x0.95mm_HandSolder, F.Cu at (129.4, 55.4)
- added C26: 4.7uF, Capacitor_SMD:C_0805_2012Metric_Pad1.18x1.45mm_HandSolder, F.Cu at (158.5, 36.6)
- added C27: 1nF/2000V, Capacitor_SMD:C_1812_4532Metric_Pad1.57x3.40mm_HandSolder, F.Cu at (164.6, 38.8)
- added C3: 0.1uF/100V, Capacitor_SMD:C_1206_3216Metric_Pad1.33x1.80mm_HandSolder, F.Cu at (163.2, 49.5)
- added C4: 15nF, Capacitor_SMD:C_0805_2012Metric_Pad1.18x1.45mm_HandSolder, F.Cu at (158.5, 27.6)
- added C6: 1nF, Capacitor_SMD:C_0603_1608Metric_Pad1.08x0.95mm_HandSolder, F.Cu at (125.1, 47.9)
- added C7: 10nF/100V, Capacitor_SMD:C_0805_2012Metric_Pad1.18x1.45mm_HandSolder, F.Cu at (158.5, 30.6)
- added C8: 27pF, Capacitor_SMD:C_0603_1608Metric_Pad1.08x0.95mm_HandSolder, F.Cu at (125.1, 50.4)
- added C9: 0.1uF, Capacitor_SMD:C_0603_1608Metric_Pad1.08x0.95mm_HandSolder, F.Cu at (125.1, 52.9)
- added D2: ABS10(LS), Diode_SMD:Diode_Bridge_Diotec_ABS, F.Cu at (162.4, 65.3)
- added D3: BAV21, Diode_SMD:D_SOD-123, F.Cu at (143.2, 60.3)
- added D4: PMEG060V100EPEZ, pi_poe:PMEG060V100EPEZ, F.Cu at (144.2, 30.4)
- added D5: SMAJ85A, Diode_SMD:D_SMA-SMB_Universal_Handsoldering, F.Cu at (97.6, 66.5)
- added D6: NC, LED_SMD:LED_0603_1608Metric_Pad1.05x0.95mm_HandSolder, F.Cu at (142.5, 66.2)
- added L1: XAL5050-103MEC, Inductor_SMD:L_Coilcraft_XAL5050-XXX, F.Cu at (136.2, 62.8)
- added R1: NC, Resistor_SMD:R_0603_1608Metric_Pad0.98x0.95mm_HandSolder, F.Cu at (129.4, 57.9)
- added R10: 10K, Resistor_SMD:R_0603_1608Metric_Pad0.98x0.95mm_HandSolder, F.Cu at (133.8, 52.9)
- added R11: 10K, Resistor_SMD:R_0603_1608Metric_Pad0.98x0.95mm_HandSolder, F.Cu at (133.8, 55.4)
- added R12: 2.49K 1%, Resistor_SMD:R_0603_1608Metric_Pad0.98x0.95mm_HandSolder, F.Cu at (133.8, 57.9)
- added R13: 510, Resistor_SMD:R_0603_1608Metric_Pad0.98x0.95mm_HandSolder, F.Cu at (138.1, 42.9)
- added R14: 510, Resistor_SMD:R_0603_1608Metric_Pad0.98x0.95mm_HandSolder, F.Cu at (138.1, 45.4)
- added R15: 10K, Resistor_SMD:R_0603_1608Metric_Pad0.98x0.95mm_HandSolder, F.Cu at (138.1, 47.9)
- added R16: 10K, Resistor_SMD:R_0603_1608Metric_Pad0.98x0.95mm_HandSolder, F.Cu at (138.1, 50.4)
- added R18: 24.9k, Resistor_SMD:R_0603_1608Metric_Pad0.98x0.95mm_HandSolder, F.Cu at (138.1, 52.9)
- added R19: 41.2, Resistor_SMD:R_0603_1608Metric_Pad0.98x0.95mm_HandSolder, F.Cu at (138.1, 55.4)
- added R2: 27K, Resistor_SMD:R_1206_3216Metric_Pad1.30x1.75mm_HandSolder, F.Cu at (163.2, 52.9)
- added R4: 51K, Resistor_SMD:R_0603_1608Metric_Pad0.98x0.95mm_HandSolder, F.Cu at (133.8, 42.9)
- added R5: 20, Resistor_SMD:R_0805_2012Metric_Pad1.20x1.40mm_HandSolder, F.Cu at (142.7, 63.4)
- added R7: 47K, Resistor_SMD:R_0603_1608Metric_Pad0.98x0.95mm_HandSolder, F.Cu at (133.8, 45.4)
- added R8: 11K, Resistor_SMD:R_0603_1608Metric_Pad0.98x0.95mm_HandSolder, F.Cu at (133.8, 47.9)
- added R9: 10K, Resistor_SMD:R_0603_1608Metric_Pad0.98x0.95mm_HandSolder, F.Cu at (133.8, 50.4)
- added T1: POE13P-50LD, pi_poe:POE13P50LD, F.Cu at (96.8, 45.7)
- added TR2: SM13126PEL, Transformer_SMD:Transformer_Ethernet_Bourns_PT61017PEL, F.Cu at (54.6, 46.0)
- added U2: MP8007GV-Z, pi_poe:MP8007GV-Z, F.Cu at (77.9, 40.7)
- added U4: RTL8152B, Package_DFN_QFN:QFN-24-1EP_4x4mm_P0.5mm_EP2.6x2.6mm, F.Cu at (101.2, 31.6)
- D1: value ABS10 -> ABS10(LS)
- moved D1 20.5 mm to (65.5, 40.1)
- moved D2 17.2 mm to (65.3, 50.0)
Connections:
- D1 pad 1: VCC -> VDD
- D1 pad 2: /VPN_IN -> VSS
- J1 pad 10: unconnected-(J1-Pad10) -> /VDD33
- J1 pad 11: unconnected-(J1-Pad11) -> Net-(J1-Pad11)
- J1 pad 12: unconnected-(J1-Pad12) -> /VDD33
- J1 pad 4: Net-(TR1-MX3+) -> PoE+_2
- J1 pad 5: Net-(TR1-MX3-) -> PoE+_2
- J1 pad 7: Net-(TR1-MX4+) -> PoE-_2
- J1 pad 8: Net-(TR1-MX4-) -> PoE-_2
- J1 pad 9: unconnected-(J1-Pad9) -> Net-(J1-Pad9)
- J1 pad SH: /VPN_IN -> unconnected-(J1-PadSH)

Commit message: pcb start
Parts:
- removed the D2 at (65.3, 50.0)
- added Y1: 25MHz, pi_poe:ABLS, F.Cu at (129.8, 104.0)
- moved C15 96.9 mm to (131.0, 122.0)
- moved J1 88.1 mm to (84.7, 124.6)
- moved D2 81.1 mm to (93.6, 108.3), turned to 180 degrees
- moved T1 79.0 mm to (115.5, 122.5)
- moved C19 77.5 mm to (101.0, 123.5), turned to -90 degrees
- moved U2 73.9 mm to (107.2, 108.5)
- moved D1 68.7 mm to (93.6, 102.8), turned to 180 degrees
- moved TR2 65.8 mm to (82.6, 105.6), turned to 90 degrees
- moved D5 32.0 mm to (107.6, 97.0)
Other:
- board outline added: 65.1 x 30.1 mm

Commit message: pcb continue
Parts:
- moved C7 115.4 mm to (43.5, 38.9), turned to 90 degrees
- moved C3 113.4 mm to (50.4, 38.8), turned to 90 degrees
- moved C15 101.9 mm to (181.0, 33.2), turned to -90 degrees
- moved D6 88.6 mm to (60.9, 32.0), turned to 90 degrees
- moved C19 88.2 mm to (88.7, 36.2)
- moved T1 84.7 mm to (127.9, 38.7)
- moved D5 84.1 mm to (46.8, 38.9), turned to -90 degrees
- moved U2 82.8 mm to (62.5, 38.9)
- moved R18 81.5 mm to (58.1, 37.5)
- moved R19 77.8 mm to (63.0, 35.0)
- moved U4 76.2 mm to (165.7, 72.2)
- moved R7 75.8 mm to (58.1, 40.4), turned to 180 degrees
- moved R1 74.6 mm to (60.9, 28.7), turned to 90 degrees
- moved C10 72.6 mm to (195.7, 72.2)
- moved C11 72.6 mm to (195.7, 74.7)
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
Commit message: pcb footprint done
Parts:
- C2, C8, Y1: moved to B.Cu
- D5: footprint Diode_SMD:D_SMA-SMB_Universal_Handsoldering -> Diode_SMD:D_SMA
- moved R14 134.9 mm to (90.1, 126.3), turned to -90 degrees
- moved R13 126.1 mm to (90.1, 102.2), turned to 90 degrees
- moved C22 122.5 mm to (128.6, 120.2), turned to 90 degrees
- moved C26 110.5 mm to (138.1, 116.0), turned to 180 degrees
- moved C15 106.7 mm to (124.7, 123.9), turned to 180 degrees
- moved D5 101.9 mm to (97.5, 127.4), turned to 180 degrees
- moved C7 101.3 mm to (97.3, 124.6), turned to 0 degrees
- moved R15 98.8 mm to (132.2, 127.1), turned to -90 degrees
- moved C3 97.5 mm to (100.6, 122.4), turned to -90 degrees
- moved C12 97.4 mm to (129.8, 127.1), turned to 180 degrees
- moved C14 96.6 mm to (121.9, 116.1), turned to 90 degrees
- moved C13 93.2 mm to (125.2, 116.1), turned to 90 degrees
- moved L1 93.1 mm to (104.9, 126.0)
- moved R16 92.8 mm to (135.2, 123.8), turned to 90 degrees
- moved R18 92.0 mm to (101.5, 118.7)
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Routing:
- net Net-(U4-CKXTAL2): track 0.00 -> 0.89 mm, vias 0 -> 1
- net Net-(U4-CKXTAL1): track 0.00 -> 0.87 mm, vias 0 -> 1

Commit message: v 1.0 of pcb almost done
Parts:
- added J2: Conn_01x04, Connector_PinHeader_2.54mm:PinHeader_1x04_P2.54mm_Vertical, F.Cu at (136.7, 128.1)
- moved Y1 29.8 mm to (121.7, 109.1)
- moved R13 27.8 mm to (111.0, 120.5), turned to 0 degrees
- moved L1 27.2 mm to (90.4, 103.1)
- moved C19 25.2 mm to (97.7, 103.2), turned to -90 degrees
- moved R11 24.6 mm to (114.7, 127.5), turned to 180 degrees
- moved R16 24.4 mm to (110.9, 126.0), turned to 0 degrees
- moved R9 24.3 mm to (114.7, 129.1), turned to 180 degrees
- moved C26 22.9 mm to (119.1, 128.8), turned to 0 degrees
- moved R10 22.4 mm to (114.5, 126.0), turned to 180 degrees
- moved R15 21.6 mm to (110.9, 123.4), turned to 0 degrees
- moved R14 20.9 mm to (110.8, 128.5), turned to 0 degrees
- moved C17 19.6 mm to (90.3, 107.9)
- moved C9 18.9 mm to (122.7, 129.0)
- moved C11 18.6 mm to (114.5, 124.4), turned to 180 degrees
- moved C8 18.4 mm to (125.9, 105.2), turned to -90 degrees
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Connections:
- J1 pad 4: PoE+_2 -> PoE-_2
- J1 pad 5: PoE+_2 -> PoE-_2
- J1 pad 7: PoE-_2 -> PoE+_2
- J1 pad 8: PoE-_2 -> PoE+_2
- T1 pad 10: GND -> Net-(D4-A_1)
- T1 pad 7: Net-(D4-A_1) -> GND
- T1 pad 8: Net-(D4-A_1) -> GND
- T1 pad 9: GND -> Net-(D4-A_1)
- TR2 pad 2: PoE+_1 -> PoE-_1
- TR2 pad 7: PoE-_1 -> PoE+_1
Routing:
- net VDD: track 0.00 -> 51.3 mm
- net Net-(D6-K): track 0.00 -> 33.5 mm, vias 0 -> 2
- net GNDD: track 0.00 -> 32.2 mm, vias 0 -> 46
- net Net-(TR2-RD+): track 0.00 -> 24.6 mm, vias 0 -> 2
- net TRANS: track 0.00 -> 21.0 mm
- net Net-(TR2-TD+): track 0.00 -> 20.6 mm, vias 0 -> 1
- net Net-(TR2-TD-): track 0.00 -> 17.5 mm, vias 0 -> 1
- net Net-(TR2-RD-): track 0.00 -> 16.7 mm, vias 0 -> 1
- net PoE-_2: track 0.00 -> 16.3 mm
- net PoE+_1: track 0.00 -> 12.9 mm
- net /VDD33: track 0.00 -> 12.4 mm
- net PoE+_2: track 0.00 -> 11.5 mm
- net +5V: track 0.00 -> 7.97 mm, vias 0 -> 2
- net /SW: track 0.00 -> 7.93 mm
- net /FB1: track 0.00 -> 7.18 mm, vias 0 -> 2
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- added copper zone on B.Cu, net GNDD
- added copper zone on F.Cu, net GNDD
- added copper zone on F.Cu, net Net-(D4-A_1)
- added copper zone on F.Cu, net TRANS
- added copper zone on F.Cu, net VDD
- added copper zone on B.Cu, net VSS
- added copper zone on F.Cu, net VSS
Other:
- board size 65.1 x 30.1 mm -> 65 x 30 mm
