File: pi_poe_hat/pi_poe_hat.kicad_pcb (KiCad board)
At the start: 2 copper layers, 65 x 30 mm, 57 parts, among them J1 8P8C_LED_Shielded, J2 Conn_01x04, T1 POE13P-50LD, U2 MP8007GV-Z, U4 RTL8152B, Y1 25MHz

Commit message: pcb almost done
Parts:
- C2, C8: moved to F.Cu
- moved R1 70.4 mm to (96.8, 133.9), turned to 180 degrees
- moved D6 66.5 mm to (100.3, 133.9), turned to 180 degrees
- moved R6 40.5 mm to (116.5, 109.2), turned to 180 degrees
- moved R3 35.1 mm to (116.5, 107.6), turned to 180 degrees
- moved R14 23.0 mm to (101.7, 115.1), turned to 0 degrees
- moved R13 18.6 mm to (101.7, 113.0), turned to 0 degrees
- moved C6 7.77 mm to (125.2, 118.8)
- moved C8 7.52 mm to (109.4, 105.8), turned to 180 degrees
- moved Y1 7.00 mm to (107.2, 107.8)
- moved R5 5.33 mm to (125.9, 115.2), turned to -90 degrees
- moved R9 4.43 mm to (113.8, 106.1)
- moved C2 3.96 mm to (99.2, 106.7)
- moved R18 1.13 mm to (104.8, 134.2)
- moved J2 0.83 mm to (120.1, 106.9)
- moved R19 0.72 mm to (102.2, 130.5)
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Connections:
- T1 pad 5: unconnected-(T1-Pad5) -> TRANS
Routing:
- net GNDD: track 0.00 -> 13.9 mm, vias 0 -> 26
- net /LED0: track 1.25 -> 10.7 mm, vias 1 -> 2
- net /LED1: track 1.20 -> 10.2 mm, vias 1 -> 2
- net Net-(U4-CKXTAL1): track 0.00 -> 8.99 mm, vias 0 -> 2
- net Net-(U4-CKXTAL2): track 0.00 -> 8.71 mm, vias 0 -> 2
- net VSS: track 0.00 -> 6.45 mm, vias 0 -> 12
- net Net-(T1-BIAS_2): track 0.00 -> 5.68 mm
- net Net-(U4-SPISD0): track 3.00 -> 8.62 mm, vias 0 -> 2
- net Net-(D6-K): track 0.00 -> 5.02 mm
- net /VDD10: track 8.34 -> 3.52 mm
- net /SW: track 0.00 -> 4.76 mm
- net /FB1: track 0.00 -> 4.07 mm
- net VDD: track 0.00 -> 3.61 mm, vias 0 -> 2
- net Net-(U4-GPIO): track 1.43 -> 4.01 mm, vias 1 -> 2
- net Net-(U2-ILIM): track 0.00 -> 2.38 mm
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- added copper zone on F.Cu, net /SW
- added copper zone on F.Cu, net GNDD
- added copper zone on F.Cu, net Net-(D3-K)
- added copper zone on F.Cu, net TRANS
- added copper zone on F.Cu, net VDD
- added copper zone on B.Cu, net VSS
- added copper zone on F.Cu, net VSS
