File: pi_poe_hat/pi_poe_hat.kicad_pcb (KiCad board)
At the start: 2 copper layers, 65 x 30 mm, 57 parts, among them J1 8P8C_LED_Shielded, J2 Conn_01x04, T1 POE13P-50LD, U2 MP8007GV-Z, U4 RTL8152B, Y1 25MHz

Commit message: second pcb done
Parts:
- moved R14 16.0 mm to (88.5, 105.8)
- moved R13 12.1 mm to (92.0, 105.8)
- moved C24 0.46 mm to (110.6, 116.5)
- moved C25 0.46 mm to (112.1, 116.5)
- moved C21 0.44 mm to (105.6, 116.5)
- moved C23 0.44 mm to (107.1, 116.5)
- moved Y1 0.25 mm to (107.2, 107.6)
- moved C20 0.23 mm to (104.2, 115.8)
- turned R15 to 180 degrees
Connections:
- T1 pad 6: unconnected-(T1-Pad6) -> GND
Routing:
- net /VDD33: track 9.06 -> 71.0 mm, vias 0 -> 7
- net +5V: track 0.00 -> 53.5 mm, vias 0 -> 1
- net /VDD10: track 3.52 -> 28.6 mm, vias 0 -> 4
- net Net-(J1-Pad9): track 0.00 -> 21.9 mm, vias 0 -> 1
- net /USB_N: track 1.00 -> 16.3 mm, vias 1 -> 2
- net /LED0: track 10.7 -> 23.9 mm
- net /USB_P: track 0.93 -> 11.8 mm, vias 1 -> 2
- net /LED1: track 10.2 -> 19.7 mm
- net Net-(J1-Pad11): track 0.00 -> 8.07 mm
- net Net-(J2-Pin_2): track 0.00 -> 6.09 mm
- net Net-(D4-A_1): track 0.00 -> 5.43 mm
- net VDD: track 3.61 -> 8.11 mm, vias 2 -> 7
- net Net-(U2-DET): track 0.00 -> 3.12 mm
- net GND: track 4.38 -> 7.35 mm, vias 0 -> 38
- net Net-(J2-Pin_1): track 0.00 -> 2.92 mm
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- added copper zone on B.Cu, net GND
- added copper zone on F.Cu, net GND
- added copper zone on B.Cu, net GNDD
- added copper zone on F.Cu, net Net-(D4-A_1)
- added copper zone on B.Cu, net VDD

Commit message: pcb done
Parts:
- moved R5 5.29 mm to (127.5, 110.2), turned to 0 degrees
- moved D4 0.32 mm to (128.9, 115.8)
- moved C6 0.05 mm to (125.2, 118.8)
Routing:
- net +5V: track 53.5 -> 12.7 mm
- net Net-(TR2-C_RX): track 0.00 -> 8.09 mm
- net Net-(C6-Pad1): track 1.95 -> 9.03 mm, vias 0 -> 2
- net GNDD: track 15.2 -> 12.6 mm
- net Net-(D4-A_1): track 5.43 -> 3.03 mm
- net /USB_P: track 11.8 -> 13.1 mm
- net Net-(T1-BIAS_2): track 5.68 -> 4.61 mm, vias 0 -> 2
- net /USB_N: track 16.3 -> 17.3 mm
- net GND: track 7.35 -> 8.02 mm, vias 38 -> 61
- net /VDD33: vias 7 -> 9
- added copper zone on F.Cu, net +5V
