File: pi_poe_hat/pi_poe_hat.kicad_sch (KiCad schematic)
At the start: 1 part, among them J1 8P8C_LED_Shielded

Commit message: pcb start
Parts:
- added TR1: SM51589PEL, Transformer_SMD:Transformer_Ethernet_Bourns_PT61020EL, symbol Transformer:PT61020EL
- added U1: PD70X01, Package_DFN_QFN:QFN-32-1EP_5x5mm_P0.5mm_EP3.3x3.3mm_ThermalVias, symbol pi_poe:PD70X01
- J1: footprint (none) -> Connector_RJ:RJ45_Amphenol_RJHSE538X
Connections:
- net at J1.1: now also TR1.23 (MX1+)
- net at J1.2: now also TR1.22 (MX1-)
- net at J1.3: now also TR1.20 (MX2+)
- net at J1.4: now also TR1.19 (MX2-)
- net at J1.5: now also TR1.17 (MX3+)
- net at J1.6: now also TR1.16 (MX3-)
- net at J1.7: now also TR1.14 (MX4+)
- net at J1.8: now also TR1.13 (MX4-)
- net GND: now reaches J1.SH
- net GND: now also U1.25 (PGND)
- new net GNDA: U1.22 (GND)
Other:
- moved on the sheet: J1

Commit message: PD done???
Parts:
- added C1: 10nF/NC, symbol Device:C
- added C10: 1uF, symbol Device:C_Small
- added C2: VAR, symbol Device:C
- added C3, C4, C5, C6: 0.01uF, symbol Device:C
- added C7: 100nF, symbol Device:C
- added C8: 1uF+, symbol Device:C
- added C9: 4.7uF, symbol Device:C_Small
- added D1, D2: ABS10, Diode_SMD:Diode_Bridge_Diotec_ABS, symbol Diode_Bridge:ABS10
- added D3, D4: LED, symbol Device:LED
- added J2: ENABLE, Connector_PinHeader_2.54mm:PinHeader_1x03_P2.54mm_Vertical, symbol Connector:Conn_01x03_Pin
- added R1, R2, R3, R4: 75, symbol Device:R
- added R10: short, symbol Device:R
- added R11, R12: 562K, symbol Device:R
- added R13: 18.7K, symbol Device:R
- added R14, R15: VAR, symbol Device:R
- added R16, R7: 24.9K, symbol Device:R
- added R17: 0, symbol Device:R_Small
- added R5, R6: 4.7K, symbol Device:R
- added R8: 240K, symbol Device:R
- added R9: 30.9K, symbol Device:R
Connections:
- net GNDA is gone; now on an unnamed net: U1.22 (GND)
- net GND: now also U1.13 (SYNC), U1.26 (CSN), U1.8 (VPN_OUT), C1.2, C2.1, C8.1, C9.1, R10.1, R10.2, R13.1, R14.1, R15.2, R16.1; no longer J1.SH
- net D4+: now reaches TR1.11 (TD4+)
- net D4-: now reaches TR1.12 (TD4-)
- net PoE+_1: now reaches TR1.15 (MCT4)
- net PoE+_1: now also C3.1, D1.4
- net at TR1.16 (MX3-): now also J1.5; no longer J1.6
- net at TR1.17 (MX3+): now also J1.4; no longer J1.5
- net PoE-_1: now reaches TR1.18 (MCT3)
- net PoE-_1: now also C4.1, D1.3
- net at TR1.19 (MX2-): now also J1.6; no longer J1.4
- net D1+: now reaches TR1.2 (TD1+)
- net PoE+_2: now reaches TR1.21 (MCT2)
- net PoE+_2: now also C5.1, D2.4
- net PoE-_2: now reaches TR1.24 (MCT1)
- net PoE-_2: now also C6.1, D2.3
- net D1-: now reaches TR1.3 (TD1-)
- net D2+: now reaches TR1.5 (TD2+)
- net D2-: now reaches TR1.6 (TD2-)
- net D3+: now reaches TR1.8 (TD3+)
- net D3-: now reaches TR1.9 (TD3-)
- net at U1.1 (RDET): now also R7.1
- net EN: now reaches U1.10 (ENABLE)
- net EN: now also J2.2 (Pin_2)
- net VINS: now reaches U1.11 (VINS)
- net VINS: now also R11.2, R12.1, R13.2
- net HYST: now reaches U1.12 (HYST)
- net HYST: now also R12.2
- net at U1.14 (RFREQ): now also R14.2
- net at U1.15 (SS): now also C2.2
- net at U1.16 (RCLP): now also R15.1
- net VL: now reaches U1.17 (VSN)
- net VL: now also U1.23 (VL), C8.2, J2.1 (Pin_1)
- net FB: now reaches U1.19 (COMP)
- net FB: now also U1.21 (FB)
- net PGOOD: now reaches U1.2 (PGOOD)
- net PGOOD: now also D3.1 (K)
- net CSP: now reaches U1.27 (CSP)
- net PG: now reaches U1.28 (PG)
- net at U1.29 (VH): now also C10.1
- net at U1.3 (RREF): now also R8.2
- net VCC: now reaches U1.30 (VCC)
- net VCC: now also U1.32 (VPP), C10.2, C7.2, C9.2, D1.1 (+), D2.1 (+), R11.1, R17.1, R5.1, R6.1, R7.2
- net at U1.31 (VAUX): now also R17.2
- net VPN_IN: now reaches U1.33 (EP)
- net VPN_IN: now also J1.SH, U1.5 (VPN_IN), C7.1, D1.2 (-), D2.2 (-), R1.2, R2.2, R3.2, R4.2, R8.1, R9.1
- net at U1.4 (RCLASS): now also R9.2
- net AT_FLAG: now reaches U1.7 (NC/AT_FLAG)
- net AT_FLAG: now also D4.1 (K)
- new net: C4.2, R2.1
- new net: C1.1, J2.3 (Pin_3)
- new net: C5.2, R3.1
- new net: C6.2, R4.1
- new net: D3.2 (A), R6.2
- new net: D4.2 (A), R5.2
- new net: C3.2, R1.1
- new net D_OUT: R16.2
- no-connect marks 0 -> 2
Other:
- note added: "BUCK"
- note added: "ENABLE"
- note added: "LED"
- note added: "PD"
- note added: "POWER"
- note added: "USB"
- note added: "UVLO"
- moved on the sheet: J1, TR1

Commit message: nothing
Parts:
- removed C1: 10nF/NC, symbol Device:C
- removed C10: 1uF, symbol Device:C_Small
- removed C2: VAR, symbol Device:C
- removed C8: 1uF+, symbol Device:C
- removed C9: 4.7uF, symbol Device:C_Small
- removed D3, D4: LED, symbol Device:LED
- removed J2: ENABLE, Connector_PinHeader_2.54mm:PinHeader_1x03_P2.54mm_Vertical, symbol Connector:Conn_01x03_Pin
- removed R10: short, symbol Device:R
- removed R11, R12: 562K, symbol Device:R
- removed R13: 18.7K, symbol Device:R
- removed R14, R15: VAR, symbol Device:R
- removed R16, R7: 24.9K, symbol Device:R
- removed R17: 0, symbol Device:R_Small
- removed R5, R6: 4.7K, symbol Device:R
- removed R8: 240K, symbol Device:R
- removed R9: 30.9K, symbol Device:R
- removed U1: PD70X01, Package_DFN_QFN:QFN-32-1EP_5x5mm_P0.5mm_EP3.3x3.3mm_ThermalVias, symbol pi_poe:PD70X01
- added C1: 1uF, symbol Device:C_Small
- added D3: 2ma, symbol Device:LED_Small
- added R18: 24.9k, symbol Device:R_Small
- added R19: 41.2, symbol Device:R_Small
- added R5: 20K, symbol Device:R_Small
- added R6: 49.9K, symbol Device:R_Small
- added R7, R8: VAR, symbol Device:R_Small
- added U1, U3: LAN7500-ABJZ, Package_DFN_QFN:QFN-56-1EP_8x8mm_P0.5mm_EP5.9x5.9mm, symbol Interface_Ethernet:LAN7500-ABJZ
- added U2: MP8007GV-Z, pi_poe:MP8007GV-Z, symbol pi_poe:MP8007GV-Z
Connections:
- net VCC: now also C1.2, R18.1, R8.1, U2.1 (AUX), U2.10 (VCC), U2.4 (VDD), U2.5 (FB2)
- net VPN_IN renamed GNDPWR
- net GNDPWR: now also R19.2, U2.23 (VSS), U2.24 (VSS), U2.25 (FTY); no longer J1.SH
- new net: R18.2, U2.2 (DET)
- new net: R7.1, U2.8 (ILIM)
- new net: D3.2 (A), R8.2
- new net: R19.1, U2.26 (CLASS)
- new net: D3.1 (K), U2.27 (T2P)
- new net: R5.1, R6.1, U2.7 (FB1)
- new net: U3.11 (VDD12CORE), U3.20 (VDD12CORE), U3.23 (VDD12CORE), U3.30 (VDD12CORE), U3.36 (VDD12CORE), U3.8 (VDD12CORE)
- new net: U3.19 (VDDVARIO), U3.24 (VDDVARIO), U3.37 (VDDVARIO), U3.7 (VDDVARIO)
- new net: U3.45 (VDD12A), U3.48 (VDD12A), U3.53 (VDD12A), U3.56 (VDD12A)
- new net C_OUT: R6.2
- new net GNDD: C1.1, R5.2, R7.2, U2.16 (GND), U2.17 (GND), U2.20 (RTN), U2.21 (RTN), U2.29, U2.6 (MODE), U2.9 (AGND)
- new net SW: U2.12 (SW), U2.13 (SW)
Other:
- note removed: "ENABLE"
- note removed: "LED"
- note removed: "UVLO"

Commit message: almost done
Parts:
- removed C3, C4, C5, C6: 0.01uF, symbol Device:C
- removed D3: 2ma, symbol Device:LED_Small
- removed R1, R2, R3, R4: 75, symbol Device:R
- removed R6: 49.9K, symbol Device:R_Small
- removed TR1: SM51589PEL, Transformer_SMD:Transformer_Ethernet_Bourns_PT61020EL, symbol Transformer:PT61020EL
- removed U1, U3: LAN7500-ABJZ, Package_DFN_QFN:QFN-56-1EP_8x8mm_P0.5mm_EP5.9x5.9mm, symbol Interface_Ethernet:LAN7500-ABJZ
- added C10, C11, C12, C25, C9: 0.1uF, symbol Device:C_Small
- added C13, C14: 47uF, symbol Device:C_Small
- added C15: 470uF, symbol Device:C_Polarized
- added C16, C17, C18: 2.2uF/100V, symbol Device:C_Small
- added C19: 47uf/100V, symbol Device:C_Polarized_Small
- added C2, C8: 27pF, symbol Device:C_Small
- added C20, C23: 0.1Uf, symbol Device:C_Small
- added C21, C24: 1uF, symbol Device:C_Small
- added C22, C26: 4.7uF, symbol Device:C_Small
- added C27: 1000p/2000V, symbol Device:C_Small
- added C3: 0.1uF/100V, symbol Device:C_Small
- added C4: 10nF, symbol Device:C_Small
- added C5: 47uF/100V, symbol Device:C_Polarized
- added C6: 1nF, symbol Device:C_Small
- added D3: BAV21, Diode_THT:D_DO-35_SOD27_P7.62mm_Horizontal, symbol Diode:BAV21
- added D4: PMEG060V100EPEZ, PMEG060V100EPEZ, symbol pi_poe:PMEG060V100EPEZ
- added D5: SMAJ85A, Diode_SMD:D_SMB, symbol Diode:SM6T18A
- added D6: NC, symbol Device:LED_Small
- added L1: XAL5050-103MEC, XAL5050103MEC, symbol pi_poe:XAL5050-103MEC
- added R1: NC, symbol Device:R_Small
- added R10, R11, R15, R16, R2, R9: 10K, symbol Device:R_Small
- added R12: 2.49K 1%, symbol Device:R_Small
- added R13, R14: 510, symbol Device:R_Small
- added R4: 91K5, symbol Device:R_Small
- added T1: POE13P-50LD, POE13P50LD, symbol pi_poe:POE13P-50LD
- added TR2: SM13126PEL, Transformer_SMD:Transformer_Ethernet_Bourns_PT61017PEL, symbol pi_poe:SM13126PEL
- added U4: RTL8152B, Package_DFN_QFN:QFN-24-1EP_4x4mm_P0.5mm_EP2.6x2.6mm, symbol pi_poe:RTL8152B
- added Y1: 25MHz, symbol Device:Crystal
- C7: value 100nF -> 10nF/100V
- D1, D2: value ABS10 -> ABS10(LS)
- R5: value 20K -> 20
- R7: value VAR -> 44K5
- R8: value VAR -> 20K
Connections:
- net D1+: now also TR2.11 (RX+), U4.4 (MDIP1)
- net D1-: now also TR2.9 (RX-), U4.5 (MDIN1)
- net GNDD: now also R8.1, C17.1, C18.1, C19.2, C27.2, T1.1 (BIAS_1); no longer R5.2
- net PoE+_1: now also TR2.2 (C_TD)
- net PoE+_2: now also J1.4, J1.5
- net PoE-_1: now also TR2.7 (C_RD)
- net PoE-_2: now also J1.7, J1.8
- net SW: now also D3.2 (A), T1.3 (PRI_1)
- net VCC: no longer C7.2, D1.1 (+), D2.1 (+), R18.1, R8.1, U2.1 (AUX), U2.4 (VDD), U2.5 (FB2)
- net FB1: now reaches R8.2
- net FB1: now also U2.7 (FB1), R4.2
- net at U2.27 (T2P): now also D6.1 (K)
- net +5V: now reaches R5.1
- net +5V: now also C13.1, C14.1, C15.1, D4.3 (K), U4.11 (VDD5); no longer U2.7 (FB1)
- net at J1.6: now also TR2.8 (RD-)
- net at J1.3: now also TR2.6 (RD+)
- net at J1.2: now also TR2.3 (TD-)
- net at J1.1: now also TR2.1 (TD+)
- net VDD33: now reaches J1.10
- net VDD33: now also J1.12, C10.2, C12.1, C22.2, C23.2, R10.2, R15.1, R16.1, R9.2, U4.1 (AVDD33), U4.10 (AVD33), U4.13 (DVDD33)
- net at J1.11: now also R13.1
- net at J1.9: now also R14.1
- net GND: now reaches J1.SH
- net GND: now also C10.1, C11.2, C12.2, C13.2, C14.2, C15.2, C2.2, C20.2, C21.2, C22.1, C23.1, C24.1, C25.1, C26.1, C27.1, C8.2, C9.1, R11.2, R12.2, T1.10 (SEC_4), T1.9 (SEC_3), U4.25 (GND), U4.6 (U2GND)
- net GNDPWR renamed VSS
- net VSS: now also C3.1, D5.2 (A2)
- new net: R15.2, U4.14 (GPIO)
- new net: C11.1, U4.16 (DVDD10)
- new net: R16.2, U4.18 (XTALDET/SPISDI)
- new net: R10.1, U4.19 (LANWAKEB)
- new net: R11.1, R9.1, U4.20 (SPISD0)
- new net: C8.1, U4.21 (CKXTAL1), Y1.2
- new net: C2.1, U4.22 (CKXTAL2), Y1.1
- new net: R12.1, U4.24 (RSET)
- new net: C6.1, R5.2
- new net: C4.2, D3.1 (K), R2.1
- new net: R4.1, T1.2 (BIAS_2)
- new net: C6.2, D4.1 (A_1), D4.2 (A_2), T1.7 (SEC_1), T1.8 (SEC_2)
- new net: D6.2 (A), R1.1
- new net: TR2.10 (C_RX), TR2.15 (C_TX)
- new net D0+: TR2.16 (TX+), U4.2 (MDIP0)
- new net D0-: TR2.14 (TX-), U4.3 (MDIN0)
- new net DVDD10: C24.2, C25.2, U4.12 (DVDD10_UPS)
- new net LED0: R14.2, U4.15 (LED0/SPICSB)
- new net LED1: R13.2, U4.17 (LED1/SPISCK)
- new net TRANS: C18.2, C19.1, C4.1, L1.2, R2.2, T1.4 (PRI_2)
- new net USB_N: U4.7 (U2DM)
- new net USB_P: U4.8 (U2DP)
- new net VDD: C17.2, C3.2, C7.2, D1.1 (+), D2.1 (+), D5.1 (A1), L1.1, R1.2, R18.1, U2.1 (AUX), U2.4 (VDD), U2.5 (FB2)
- new net VDD10: C20.1, C21.1, C26.2, C9.2, U4.23 (AVDD10), U4.9 (U2VDD10)
- no-connect marks 2 -> 4
Other:
- note added: "Choke"
- note removed: "POWER"
- moved on the sheet: C1, C7, D1, J1, R18, R19, R7, U2

Commit message: done?
Parts:
- removed C16: 2.2uF/100V, symbol Device:C_Small
- removed C5: 47uF/100V, symbol Device:C_Polarized
- C1, C10, C11, C12, C2, C20, C21, C23, C24, C25, C6, C8, C9: footprint (none) -> Capacitor_SMD:C_0603_1608Metric_Pad1.08x0.95mm_HandSolder
- C13, C14, C17, C18: footprint (none) -> Capacitor_SMD:C_1210_3225Metric_Pad1.33x2.70mm_HandSolder
- C15: value 470uF -> 470uF/16V; footprint (none) -> Capacitor_THT:CP_Radial_D10.0mm_P5.00mm
- C19: footprint (none) -> Capacitor_THT:CP_Radial_D8.0mm_P3.50mm
- C22, C26, C7: footprint (none) -> Capacitor_SMD:C_0805_2012Metric_Pad1.18x1.45mm_HandSolder
- C27: value 1000p/2000V -> 1nF/2000V; footprint (none) -> Capacitor_SMD:C_1812_4532Metric_Pad1.57x3.40mm_HandSolder
- C3: footprint (none) -> Capacitor_SMD:C_1206_3216Metric_Pad1.33x1.80mm_HandSolder
- C4: value 10nF -> 15nF; footprint (none) -> Capacitor_SMD:C_0805_2012Metric_Pad1.18x1.45mm_HandSolder
- D3: footprint Diode_THT:D_DO-35_SOD27_P7.62mm_Horizontal -> Diode_SMD:D_SOD-123
- D4: footprint PMEG060V100EPEZ -> pi_poe:PMEG060V100EPEZ
- D5: footprint Diode_SMD:D_SMB -> Diode_SMD:D_SMA-SMB_Universal_Handsoldering
- D6: footprint (none) -> LED_SMD:LED_0603_1608Metric_Pad1.05x0.95mm_HandSolder
- L1: footprint XAL5050103MEC -> Inductor_SMD:L_Coilcraft_XAL5050-XXX
- R1, R10, R11, R12, R13, R14, R15, R16, R18, R19, R9: footprint (none) -> Resistor_SMD:R_0603_1608Metric_Pad0.98x0.95mm_HandSolder
- R2: value 10K -> 27K; footprint (none) -> Resistor_SMD:R_1206_3216Metric_Pad1.30x1.75mm_HandSolder
- R4: value 91K5 -> 51K; footprint (none) -> Resistor_SMD:R_0603_1608Metric_Pad0.98x0.95mm_HandSolder
- R5: footprint (none) -> Resistor_SMD:R_0805_2012Metric_Pad1.20x1.40mm_HandSolder
- R7: value 44K5 -> 47K; footprint (none) -> Resistor_SMD:R_0603_1608Metric_Pad0.98x0.95mm_HandSolder
- R8: value 20K -> 11K; footprint (none) -> Resistor_SMD:R_0603_1608Metric_Pad0.98x0.95mm_HandSolder
- T1: footprint POE13P50LD -> pi_poe:POE13P50LD
Connections:
- net GND: no longer J1.SH
- no-connect marks 4 -> 5
Other:
- note added: "ETH"
- moved on the sheet: C1, C10, C11, C12, C13, C14, C15, C17, C18, C19, C2, C20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

Commit message: pcb start
Parts:
- Y1: footprint (none) -> pi_poe:ABLS
Changed lines of the file:
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@@
       (effects (font (size 1.27 1.27)))
     )
-    (property "Footprint" "" (at 189.23 125.73 0)
+    (property "Footprint" "pi_poe:ABLS" (at 189.23 125.73 0)
       (effects (font (size 1.27 1.27)) hide)
     )

Commit message: pcb footprint done
Parts:
- D5: footprint Diode_SMD:D_SMA-SMB_Universal_Handsoldering -> Diode_SMD:D_SMA
Changed lines of the file:
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@@
       (effects (font (size 1.27 1.27)) (justify left))
     )
-    (property "Footprint" "Diode_SMD:D_SMA-SMB_Universal_Handsoldering" (at 78.74 43.18 0)
+    (property "Footprint" "Diode_SMD:D_SMA" (at 78.74 43.18 0)
       (effects (font (size 1.27 1.27)) hide)
     )

Commit message: v 1.0 of pcb almost done
Parts:
- added J2: Conn_01x04, Connector_PinHeader_2.54mm:PinHeader_1x04_P2.54mm_Vertical, symbol Connector_Generic:Conn_01x04
- added R3, R6: 0, Resistor_SMD:R_0603_1608Metric_Pad0.98x0.95mm_HandSolder, symbol Device:R_Small
Connections:
- net +5V: now also J2.3 (Pin_3)
- net GND: now also T1.7 (SEC_1), T1.8 (SEC_2), J2.4 (Pin_4); no longer T1.10 (SEC_4), T1.9 (SEC_3)
- net PoE+_1: now also TR2.7 (C_RD); no longer TR2.2 (C_TD)
- net PoE+_2: now also J1.7, J1.8; no longer J1.4, J1.5
- net PoE-_1: now also TR2.2 (C_TD); no longer TR2.7 (C_RD)
- net PoE-_2: now also J1.4, J1.5; no longer J1.7, J1.8
- net USB_N: now also R3.2
- net USB_P: now also R6.2
- net at C6.2, D4.1 (A_1), D4.2 (A_2): now also T1.10 (SEC_4), T1.9 (SEC_3); no longer T1.7 (SEC_1), T1.8 (SEC_2)
- new net: J2.1 (Pin_1), R3.1
- new net: J2.2 (Pin_2), R6.1
Other:
- moved on the sheet: C13, C14, C15, C6, D4, R5
