File: pi_poe_hat/pi_poe_hat.kicad_sch (KiCad schematic)
At the start: 57 parts, among them J1 8P8C_LED_Shielded, J2 Conn_01x04, T1 POE13P-50LD, U2 MP8007GV-Z, U4 RTL8152B, Y1 25MHz

Commit message: second pcb almost done
Connections:
- net GNDD: now also U2.11 (N/C), U2.14 (N/C), U2.15 (N/C), U2.19 (N/C), U2.22 (N/C), U2.28 (N/C), U2.3 (N/C)
- net PoE+_1: now also TR2.2 (C_TD); no longer TR2.7 (C_RD)
- net PoE-_1: now also TR2.7 (C_RD); no longer TR2.2 (C_TD)
