File: pi_poe_hat/pi_poe_hat_backup.kicad_pcb (KiCad board)
At the start: 2 copper layers, 65 x 30 mm, 57 parts, among them J1 8P8C_LED_Shielded, J2 Conn_01x04, T1 POE13P-50LD, U2 MP8007GV-Z, U4 RTL8152B, Y1 25MHz

Commit message: second pcb almost done
Parts:
- C27: moved to F.Cu
- moved R3 62.1 mm to (133.2, 129.1), turned to 180 degrees
- moved R6 62.0 mm to (126.6, 129.1), turned to 180 degrees
- moved D6 51.3 mm to (75.4, 106.6)
- moved R1 51.3 mm to (75.4, 103.1)
- moved R13 33.6 mm to (110.8, 125.5), turned to 0 degrees
- moved R14 32.8 mm to (111.0, 120.7), turned to 0 degrees
- moved C9 29.6 mm to (122.7, 129.0), turned to 180 degrees
- moved C26 28.6 mm to (119.1, 128.8)
- moved R12 28.1 mm to (123.4, 127.4), turned to 0 degrees
- moved J2 27.5 mm to (136.7, 128.1), turned to 180 degrees
- moved C2 26.7 mm to (125.9, 113.1)
- moved C10 25.8 mm to (123.5, 124.8), turned to -90 degrees
- moved D2 23.9 mm to (81.2, 105.2), turned to -90 degrees
- moved R9 23.5 mm to (114.2, 129.1), turned to 180 degrees
- moved R11 23.0 mm to (114.2, 127.5)
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Connections:
- TR2 pad 2: PoE+_1 -> PoE-_1
- TR2 pad 7: PoE-_1 -> PoE+_1
Routing:
- net VDD: track 0.00 -> 51.3 mm
- net +5V: track 0.00 -> 33.8 mm, vias 0 -> 2
- net GNDD: track 0.00 -> 32.2 mm, vias 0 -> 46
- net D1-: track 8.30 -> 37.2 mm
- net D1+: track 12.0 -> 35.2 mm
- net TRANS: track 0.00 -> 21.0 mm
- net D0-: track 15.8 -> 33.2 mm
- net /USB_N: track 0.00 -> 14.9 mm, vias 0 -> 2
- net D0+: track 18.5 -> 32.0 mm
- net /VDD33: track 9.40 -> 22.1 mm
- net /USB_P: track 0.00 -> 12.0 mm
- net Net-(J2-Pin_2): track 0.00 -> 10.7 mm
- net PoE+_2: track 21.6 -> 11.5 mm
- net Net-(TR2-TD+): track 11.8 -> 20.6 mm, vias 0 -> 1
- net PoE+_1: track 4.49 -> 12.9 mm
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- added copper zone on B.Cu, net GNDD
- added copper zone on F.Cu, net GNDD
- added copper zone on F.Cu, net Net-(D4-A_1)
- added copper zone on F.Cu, net TRANS
- added copper zone on F.Cu, net VDD
- added copper zone on B.Cu, net VSS
- added copper zone on F.Cu, net VSS
Other:
- outline, holes or cut-outs redrawn
